Commit message: a1 urdf fixed

File: robots/a1/arcus_1.5_4.urdf (robot description, URDF)
Before this commit: robot arcus_1.5_4, 24 links, 23 joints
Links:
- added link world
- link left_ankle_pitch_link: mass 0.0267996226956392 -> 0.0267996226956345
- link left_ankle_roll_link: mass 0.661703325569247 -> 0.661563785020683
- link left_elbow_link: mass 0.793513817454599 -> 0.79351383141003
- link left_hip_pitch_link: mass 1.39230542107987 -> 1.39230705559468
- link left_hip_roll_link: mass 1.47113347070104 -> 1.4711381233483
- link left_hip_yaw_link: mass 1.70259905291502 -> 1.70259926154147
- link left_knee_link: mass 2.19047791510296 -> 2.19039898991067
- link left_shoulder_pitch_link: mass 0.856999833939349 -> 0.856999831581915
- link left_shoulder_roll_link: mass 0.576808851401746 -> 0.57680884793817
- link left_shoulder_yaw_link: mass 0.787455808914453 -> 0.787456261562816
- link right_ankle_pitch_link: mass 0.0267996226956392 -> 0.0267996226956345
- link right_ankle_roll_link: mass 0.661703325569247 -> 0.661563785020683
- link right_elbow_link: mass 0.793513817454599 -> 0.79351383141003
- link right_hip_pitch_link: mass 1.39230542107987 -> 1.39230705559468
- link right_hip_roll_link: mass 1.47113347070104 -> 1.4711381233483
- link right_hip_yaw_link: mass 1.70259905291502 -> 1.70259926154147
- link right_knee_link: mass 2.19047791510296 -> 2.19039898991067
- link right_shoulder_pitch_link: mass 0.856999833939349 -> 0.856999831581915
- link right_shoulder_roll_link: mass 0.576808851401746 -> 0.57680884793817
- link right_shoulder_yaw_link: mass 0.787455808914453 -> 0.787456261562816
- link right_wrist_roll_rubber_hand: mass 0.278928121537221 -> 0.278919926883193
Joints:
- added joint floating_base_joint: type floating, parent world, child pelvis

Commit message: a1 urdf fixed

File: robots/a1/arcus_1.5_4.urdf (robot description, URDF)
Before this commit: robot arcus_1.5_3, 24 links, 23 joints
Links:
- link left_ankle_pitch_link: mass 0.0267996226956345 -> 0.0267996226956392
- link left_ankle_roll_link: mass 0.661563785020683 -> 0.661703325569247
- link left_elbow_link: mass 0.79351383141003 -> 0.793513817454599
- link left_hip_pitch_link: mass 1.39230705559468 -> 1.39230542107987
- link left_hip_roll_link: mass 1.4711381233483 -> 1.47113347070104
- link left_hip_yaw_link: mass 1.70259926154147 -> 1.70259905291502
- link left_knee_link: mass 2.19039898991067 -> 2.19047791510296
- link left_shoulder_pitch_link: mass 0.856999831581915 -> 0.856999833939349
- link left_shoulder_roll_link: mass 0.57680884793817 -> 0.576808851401746
- link left_shoulder_yaw_link: mass 0.787456261562816 -> 0.787455808914453
- link right_ankle_pitch_link: mass 0.0267996226956345 -> 0.0267996226956392
- link right_ankle_roll_link: mass 0.661563785020683 -> 0.661703325569247
- link right_elbow_link: mass 0.79351383141003 -> 0.793513817454599
- link right_hip_pitch_link: mass 1.39230705559468 -> 1.39230542107987
- link right_hip_roll_link: mass 1.4711381233483 -> 1.47113347070104
- link right_hip_yaw_link: mass 1.70259926154147 -> 1.70259905291502
- link right_knee_link: mass 2.19039898991067 -> 2.19047791510296
- link right_shoulder_pitch_link: mass 0.856999831581915 -> 0.856999833939349
- link right_shoulder_roll_link: mass 0.57680884793817 -> 0.576808851401746
- link right_shoulder_yaw_link: mass 0.787456261562816 -> 0.787455808914453
- link right_wrist_roll_rubber_hand: mass 0.278919926883193 -> 0.278928121537221
