Commit message: arcus urdf and mechanical fixing

File: robots/a1/arcus_1.5_6.urdf (robot description, URDF)
Before this commit: robot arcus_1.5_5, 24 links, 23 joints
Links:
- link left_elbow_link: mass 0.793513817454599 -> 0.6; geometry visual mesh filename=meshes/left_elbow_link.STL
- link left_shoulder_pitch_link: mass 0.856999833939349 -> 0.718
- link left_shoulder_roll_link: mass 0.576808851401746 -> 0.643
- link left_shoulder_yaw_link: mass 0.787455808914453 -> 0.734
- link pelvis: mass 4.806 -> 3.813; geometry visual mesh filename=meshes/pelvis.STL
- link right_elbow_link: mass 0.793513817454599 -> 0.6; geometry visual mesh filename=meshes/right_elbow_link.STL
- link right_shoulder_pitch_link: mass 0.856999833939349 -> 0.718
- link right_shoulder_roll_link: mass 0.576808851401746 -> 0.643
- link right_shoulder_yaw_link: mass 0.787455808914453 -> 0.734
