Commit message: arcus a2 long step reward fixing, urdf fixing

File: robots/arcus/a2/a2_12.urdf (robot description, URDF)
Before this commit: robot a2_12, 15 links, 14 joints
Links:
- link left_ankle_roll_link: mass 0.521206684966548 -> 0.522
- link left_hip_pitch_link: mass 1.13692961688961 -> 1.137
- link left_hip_roll_link: mass 1.11015839475992 -> 1.11015
- link left_hip_yaw_link: mass 0.915775189402335 -> 0.92
- link left_knee_link: mass 1.07153118596826 -> 1.07
- link right_ankle_roll_link: mass 0.52126220426659 -> 0.522
- link right_hip_pitch_link: mass 1.13717442710025 -> 1.137
- link right_hip_roll_link: mass 1.11015680631126 -> 1.11015
- link right_hip_yaw_link: mass 0.915775178235333 -> 0.92
- link right_knee_link: mass 1.07142387779233 -> 1.07
