Commit message: arcus 2 IL env added

File: robots/arcus/a2/acrus2_v0.urdf (robot description, URDF)
Before this commit: robot acrus2_v0, 15 links, 14 joints
Joints:
- joint waist_yaw_joint: type fixed -> revolute

File: robots/arcus/a2/acrus2_v0_23.urdf (robot description, URDF)
Before this commit: robot a2_12, 15 links, 14 joints
Links:
- added link left_elbow_link
- added link left_shoulder_pitch_link
- added link left_shoulder_roll_link
- added link left_shoulder_yaw_link
- added link left_wrist_roll_link
- added link right_elbow_link
- added link right_shoulder_pitch_link
- added link right_shoulder_roll_link
- added link right_shoulder_yaw_link
- added link right_wrist_roll_link
- link left_ankle_pitch_link: mass 0.026795 -> 0.039555
- link left_ankle_roll_link: mass 0.522 -> 0.55367
- link left_hip_pitch_link: mass 1.137 -> 1.1042
- link left_hip_roll_link: mass 1.11015 -> 1.4731
- link left_hip_yaw_link: mass 0.92 -> 1.6219
- link left_knee_link: mass 1.07 -> 1.8088
- link pelvis: mass 1.14864897245035 -> 3.7759
- link right_ankle_pitch_link: mass 0.026795 -> 0.039555
- link right_ankle_roll_link: mass 0.522 -> 0.55367
- link right_hip_pitch_link: mass 1.137 -> 1.1042
- link right_hip_roll_link: mass 1.11015 -> 1.4731
- link right_hip_yaw_link: mass 0.92 -> 1.6219
- link right_knee_link: mass 1.07 -> 1.8088
- link torso_link: mass 3.598 -> 5.3141
Joints:
- added joint left_elbow_joint: type revolute, parent torso_link, child left_elbow_link, origin xyz=0 0 0.0 rpy=0 0 0
- added joint left_shoulder_pitch_joint: type revolute, parent torso_link, child left_shoulder_pitch_link, origin xyz=0 0 0.0 rpy=0 0 0
- added joint left_shoulder_roll_joint: type revolute, parent torso_link, child left_shoulder_roll_link, origin xyz=0 0 0.0 rpy=0 0 0
- added joint left_shoulder_yaw_joint: type revolute, parent torso_link, child left_shoulder_yaw_link, origin xyz=0 0 0.0 rpy=0 0 0
- added joint left_wrist_roll_joint: type revolute, parent torso_link, child left_wrist_roll_link, origin xyz=0 0 0.0 rpy=0 0 0
- added joint right_elbow_joint: type revolute, parent torso_link, child right_elbow_link, origin xyz=0 0 0.0 rpy=0 0 0
- added joint right_shoulder_pitch_joint: type revolute, parent torso_link, child right_shoulder_pitch_link, origin xyz=0 0 0.0 rpy=0 0 0
- added joint right_shoulder_roll_joint: type revolute, parent torso_link, child right_shoulder_roll_link, origin xyz=0 0 0.0 rpy=0 0 0
- added joint right_shoulder_yaw_joint: type revolute, parent torso_link, child right_shoulder_yaw_link, origin xyz=0 0 0.0 rpy=0 0 0
- added joint right_wrist_roll_joint: type revolute, parent torso_link, child right_wrist_roll_link, origin xyz=0 0 0.0 rpy=0 0 0
- joint left_ankle_pitch_joint: origin xyz=0.0051571 0.0038133 -0.34537 rpy=0 0 0 -> xyz=0.0051382 -0.0061861 -0.34527 rpy=0 0 0
- joint left_ankle_roll_joint: origin xyz=-0.036853 -0.019526 -0.010727 rpy=0 0 0 -> xyz=-0.028834 -0.0095267 -0.010835 rpy=0 0 0
- joint left_hip_roll_joint: origin xyz=0.039629 0.053649 -0.02998 rpy=0 0 0 -> xyz=0.038629 0.053649 -0.02998 rpy=0 0 0
- joint left_hip_yaw_joint: origin xyz=-0.039847 0.00013269 -0.12033 rpy=0 0 0 -> xyz=-0.038847 0.00013269 -0.12033 rpy=0 0 0
- joint right_ankle_pitch_joint: origin xyz=0.0051571 -0.0030667 -0.34537 rpy=0 0 0 -> xyz=0.0051382 0.0069327 -0.34527 rpy=0 0 0
- joint right_ankle_roll_joint: origin xyz=-0.036853 0.019526 -0.010727 rpy=0 0 0 -> xyz=-0.028834 0.0095267 -0.010835 rpy=0 0 0
- joint right_knee_joint: limit lower=-0.1 upper=2.9 effort=130 velocity=20 -> lower=-0.1 upper=2.9 effort=130 velocity=31
- joint waist_yaw_joint: type fixed -> revolute
