Commit message: env fixing

File: robots/arcus/a2/acrus2_v0_29.urdf (robot description, URDF)
Before this commit: robot acrus2_v0, 31 links, 30 joints
Links:
- link left_ankle_roll_link: geometry collision sphere radius=0.005; collision sphere radius=0.005
- link pelvis: geometry visual mesh filename=meshes/pelvis.STL
- link right_ankle_roll_link: geometry collision sphere radius=0.005; collision sphere radius=0.005
