Commit message: URDF/mjcfg fixed, IL fixed

File: robots/arcus/a2/acrus2_v1_23.urdf (robot description, URDF)
Before this commit: robot acrus2_v0, 25 links, 24 joints
Joints:
- joint left_hip_roll_joint: limit lower=-0.5 upper=2 effort=130 velocity=31 -> lower=-0.362 upper=2 effort=130 velocity=31
- joint left_knee_joint: limit lower=-0.1 upper=2.9 effort=130 velocity=31 -> lower=-0.1 upper=2.52 effort=130 velocity=31
- joint right_hip_roll_joint: limit lower=-2 upper=0.5 effort=130 velocity=31 -> lower=-2 upper=0.362 effort=130 velocity=31
- joint right_knee_joint: limit lower=-0.1 upper=2.9 effort=130 velocity=31 -> lower=-0.1 upper=2.52 effort=130 velocity=31
