Commit message: standing up congif added; walking config reward fixed

File: robots/arcus/a1_2/Arcus_2_original_arms29.urdf (robot description, URDF)
Before this commit: robot Arcus2.SLDASM, 34 links, 33 joints
Links:
- link left_knee_link: geometry collision mesh filename=meshes/left_knee_link.STL; visual mesh filename=meshes/left_knee_link.STL
- link right_knee_link: geometry collision mesh filename=meshes/right_knee_link.STL; visual mesh filename=meshes/right_knee_link.STL
