Commit message: cart fixed

File: cart/cart.urdf (robot description, URDF)
Before this commit: robot multi_level_profile_cart, 14 links, 13 joints
Joints:
- joint arm_left_joint: origin xyz=-0.22 0.2 0 rpy=-0.785398 0 1.57079632679 -> xyz=-0.22 0.2 0.1 rpy=-0.785398 0 1.57079632679
- joint arm_right_joint: origin xyz=-0.22 -0.2 0 rpy=0.785398 0 -1.57079632679 -> xyz=-0.22 -0.2 0.1 rpy=0.785398 0 -1.57079632679
